File: pcbproject/altsdr_rf_board/altsdr_rf_board.sch (KiCad schematic (older format))
At the start: 3 parts

Commit message: schematic work + more libs
Parts:
- added J?: CX70M-24P1, digikey-footprints:USB-C_Female_CX70M-24P1, symbol dk_USB-DVI-HDMI-Connectors:CX70M-24P1
- added J? (x3): 5-1814400-1, digikey-footprints:RF_SMA_RightAngle_5-1814400-1, symbol dk_Coaxial-Connectors-RF:5-1814400-1
- added R? (x2): 5.1k, RESC2012X65N, symbol 9-2176091-2:9-2176091-2
- added U?: MAX3523ETP+, QFN65P500X500X80-21N, symbol MAX3523ETP_:MAX3523ETP+
- added U? (x2): Si514, symbol Si514:Si514
- added U? (x2): pe4140b, symbol pe4140b:pe4140b
- added U?: AP2114H-3_3TRG1, digikey-footprints:SOT-223, symbol dk_PMIC-Voltage-Regulators-Linear:AP2114H-3_3TRG1
- added U? (x10): SKY13414-485LF, IC_SKY13414-485LF, symbol SKY13414-485LF:SKY13414-485LF
Connections:
- net at U?.100 (PA11): now also J?.A7, J?.B7
- net at U?.101 (PA12): now also J?.A6, J?.B6
- net at U?.133 (PB6): now also U?.2 (SCL), U?.2 (SCL), U?.6 (SCLK)
- net at U?.134 (PB7): now also U?.1 (SDA), U?.1 (SDA), U?.7 (SDA)
- net at U?.39 (PA2): now also U?.6 (IF2)
- net at U?.40 (PA3): now also U?.1 (IF1)
- net at U?.43 (PA4): now also U?.1 (IF1)
- net at U?.44 (PA5): now also U?.6 (IF2)
- net at U?.104 (VSS): now also U?.118 (VSS), U?.12 (VSS), U?.128 (VSS), U?.141 (VSS), U?.18 (VSS), U?.33 (VSS), U?.41 (VSS), U?.55 (VSS), U?.6 (VSS), U?.69 (VSS), U?.80 (VSS), U?.89 (VSS)
- net at U?.106 (VDD): now also U?.119 (VDD), U?.129 (VDD), U?.13 (VDD), U?.144 (VDD), U?.19 (VDD), U?.32 (VDD), U?.42 (VDD), U?.56 (VDD), U?.7 (VDD), U?.71 (VDD), U?.79 (VDD), U?.92 (VDD)
- new net: U?.12 (OUT-), U?.13 (ANT)
- new net: U?.13 (ANT), U?.14 (OUT+)
- new net: U?.2 (IN+), U?.2 (RF1)
- new net: U?.3 (IN-), U?.3 (RF2)
- new net: U?.4 (CLK+), U?.5 (LO1) (x2)
- new net: U?.4 (LO2), U?.5 (CLK-) (x2)
- new net: U?.13 (ANT), U?.2 (RF1)
- new net: U?.13 (ANT), U?.3 (RF2)
- new net: J?.A4, J?.A9, J?.B4, J?.B9, U?.3 (IN)
- new net: J?.A1, J?.B12, R?.1
- new net: J?.A12, J?.B1, R?.2
- new net: J?.A5, R?.2
- new net: J?.B5, R?.1
- new net: U?.10 (RF4), U?.9 (RF2) (x2)
- new net: U?.2 (RF3), U?.9 (RF2) (x2)
- new net: U?.9 (RF2), U?.9 (RF2) (x2)
- new net: U?.10 (RF4), U?.3 (RF1) (x2)
- new net: U?.2 (RF3), U?.3 (RF1) (x2)
- new net: U?.3 (RF1), U?.9 (RF2) (x2)
- new net: J?.1, U?.13 (ANT) (x2)
- new net: J?.2, U?.13 (ANT) (x3)
- new net: J?.1, U?.4 (VDD)
Other:
- moved on the sheet: U?B, U?C

Commit message: add power ports to schematic
Parts:
- added P? (x16): GND_, symbol power_ports:GND_
- added P?: +5v, symbol power_ports:+5v
- added P?: +3v, symbol power_ports:+3v
Connections:
- net at U?.104 (VSS), U?.118 (VSS), U?.12 (VSS)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: now also P?.~
- net at U?.1 (GND-2): now also U?.18 (GND-1), U?.5 (GND), P?.~
- net at U?.10 (VDD-1): now also U?.17 (VDD)
- net at U?.3 (GND): now also P?.~ (x2)
- net at U?.1 (GND): now also P?.~
- net at U?.2 (VOUT): now also U?.4 (VOUT), P?.~
- net at J?.A4, J?.A9, J?.B4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: now also P?.~
- net at J?.A1, J?.B12, R?.1: now also P?.~
- net at J?.A12, J?.B1, R?.2: now also P?.~
- net at U?.15 (GND): now also P?.~ (x9)
Changed lines of the file:
@@
 Connection ~ 16550 1550
 Wire Wire Line
-	16550 1550 16550 1650
+	16550 1550 16550 1600
 Connection ~ 16550 1650
 Wire Wire Line
@@
 Wire Wire Line
 	700  1700 1200 1700
-$Comp
-L MAX3523ETP_:MAX3523ETP+ U?
-U 1 1 5FEA0D8A
-P 8250 6450
-F 0 "U?" H 8250 7820 50  0000 C CNN
-F 1 "MAX3523ETP+" H 8250 7729 50  0000 C CNN
-F 2 "QFN65P500X500X80-21N" H 8250 6450 50  0001 L BNN
-F 3 "" H 8250 6450 50  0001 L BNN
-F 4 "QFN65P500X500X80-21N" H 8250 6450 50  0001 L BNN "Package"
-F 5 "Maxim Integrated" H 8250 6450 50  0001 L BNN "Manufacturer"
-	1    8250 6450
-	1    0    0    -1
-$EndComp
 $Comp
 L Si514:Si514 U?
@@
 $EndComp
 Wire Wire Line
-	7550 5650 7550 4800
-Wire Wire Line
-	7550 4800 4950 4800
-Wire Wire Line
 	4950 4800 4950 5450
 Wire Wire Line
@@
 Wire Wire Line
 	4900 5600 4900 4750
-Wire Wire Line
-	4900 4750 7500 4750
-Wire Wire Line
-	7500 4750 7500 5750
 Wire Wire Line
 	7500 5750 7550 5750
@@
 	19700 4750 19700 4200
 Wire Wire Line
-	19700 4200 20700 4200
+	19700 4200 20250 4200
 Wire Wire Line
 	20700 4200 20700 4550
@@
 	20700 5850 20700 6500
 Wire Wire Line
-	20700 6500 19400 6500
+	20700 6500 20100 6500
 Wire Wire Line
 	19400 6500 19400 5850
@@
 Wire Wire Line
 	15550 17800 16800 17800
+$Comp
+L power_ports:GND_ P?
+U 1 1 5FE1536B
+P 16750 1600
+F 0 "P?" V 16704 1528 50  0000 L CNN
+F 1 "GND_" V 16795 1528 50  0000 L CNN
+F 2 "" H 16750 1650 50  0001 C CNN
+F 3 "" H 16750 1650 50  0001 C CNN
+	1    16750 1600
+	0    1    1    0
+$EndComp
+Connection ~ 16550 1600
+Wire Wire Line
+	16550 1600 16550 1650
+$Comp
+L power_ports:GND_ P?
+U 1 1 5FE1E507
+P 20100 6700
+F 0 "P?" H 19972 6496 50  0000 R CNN
+F 1 "GND_" H 19972 6587 50  0000 R CNN
+F 2 "" H 20100 6750 50  0001 C CNN
+F 3 "" H 20100 6750 50  0001 C CNN
+	1    20100 6700
+	-1   0    0    1
+$EndComp
+Connection ~ 20100 6500
+Wire Wire Line
+	20100 6500 19400 6500
+$Comp
+L power_ports:GND_ P?
+U 1 1 5FE21E03
+P 20250 4000
+F 0 "P?" H 20378 3889 50  0000 L CNN
+F 1 "GND_" H 20378 3798 50  0000 L CNN
+F 2 "" H 20250 4050 50  0001 C CNN
+F 3 "" H 20250 4050 50  0001 C CNN
+	1    20250 4000
+	1    0    0    -1
+$EndComp
+Connection ~ 20250 4200
+Wire Wire Line
+	20250 4200 20700 4200
+$Comp
+L power_ports:+5v P?
+U 1 1 5FE2D177
+P 17100 7300
+F 0 "P?" V 17365 7017 50  0000 C CNN
+F 1 "+5v" V 17274 7017 50  0000 C CNN
+F 2 "" H 17100 7300 50  0001 C CNN
+F 3 "" H 17100 7300 50  0001 C CNN
+	1    17100 7300
+	0    -1   -1   0
+$EndComp
+Connection ~ 17450 7300
+Wire Wire Line
+	18350 6500 18350 6550
+$Comp
+L power_ports:GND_ P?
+U 1 1 5FE3AB67
+P 17850 7200
+F 0 "P?" H 17722 6996 50  0000 R CNN
+F 1 "GND_" H 17722 7087 50  0000 R CNN
+F 2 "" H 17850 7250 50  0001 C CNN
+F 3 "" H 17850 7250 50  0001 C CNN
+	1    17850 7200
+	-1   0    0    1
+$EndComp
+$Comp
+L power_ports:+3v P?
+U 1 1 5FE3BBBE
+P 18700 6550
+F 0 "P?" V 18654 6378 50  0000 L CNN
+F 1 "+3v" V 18745 6378 50  0000 L CNN
+F 2 "" H 18700 6550 50  0001 C CNN
+F 3 "" H 18700 6550 50  0001 C CNN
+	1    18700 6550
+	0    1    1    0
+$EndComp
+Connection ~ 18350 6550
+Wire Wire Line
+	18350 6550 18350 6600
+$Comp
+L power_ports:GND_ P?
+U 1 1 5FE42EBF
+P 18300 13400
+F 0 "P?" V 18254 13328 50  0000 L CNN
+F 1 "GND_" V 18345 13328 50  0000 L CNN
+F 2 "" H 18300 13450 50  0001 C CNN
+F 3 "" H 18300 13450 50  0001 C CNN
+	1    18300 13400
+	0    1    1    0
+$EndComp
+$Comp
+L power_ports:GND_ P?
+U 1 1 5FE457D8
+P 18250 14850
+F 0 "P?" V 18204 14778 50  0000 L CNN
+F 1 "GND_" V 18295 14778 50  0000 L CNN
+F 2 "" H 18250 14900 50  0001 C CNN
+F 3 "" H 18250 14900 50  0001 C CNN
+	1    18250 14850
+	0    1    1    0
+$EndComp
+$Comp
+L power_ports:GND_ P?
+U 1 1 5FE5E633
+P 18200 11450
+F 0 "P?" V 18154 11378 50  0000 L CNN
+F 1 "GND_" V 18245 11378 50  0000 L CNN
+F 2 "" H 18200 11500 50  0001 C CNN
+F 3 "" H 18200 11500 50  0001 C CNN
+	1    18200 11450
+	0    1    1    0
+$EndComp
+$Comp
+L power_ports:GND_ P?
+U 1 1 5FE75B91
+P 18250 10000
+F 0 "P?" V 18204 9928 50  0000 L CNN
+F 1 "GND_" V 18295 9928 50  0000 L CNN
+F 2 "" H 18250 10050 50  0001 C CNN
+F 3 "" H 18250 10050 50  0001 C CNN
+	1    18250 10000
+	0    1    1    0
+$EndComp
+$Comp
+L power_ports:GND_ P?
+U 1 1 5FE82CDD
+P 18250 17050
+F 0 "P?" V 18204 16978 50  0000 L CNN
+F 1 "GND_" V 18295 16978 50  0000 L CNN
+F 2 "" H 18250 17100 50  0001 C CNN
+F 3 "" H 18250 17100 50  0001 C CNN
+	1    18250 17050
+	0    1    1    0
+$EndComp
+$Comp
+L power_ports:GND_ P?
+U 1 1 5FE8DCA6
+P 18200 18500
+F 0 "P?" V 18154 18428 50  0000 L CNN
+F 1 "GND_" V 18245 18428 50  0000 L CNN
+F 2 "" H 18200 18550 50  0001 C CNN
+F 3 "" H 18200 18550 50  0001 C CNN
+	1    18200 18500
+	0    1    1    0
+$EndComp
+$Comp
+L power_ports:GND_ P?
+U 1 1 5FEA22F7
+P 6400 11000
+F 0 "P?" V 6354 10928 50  0000 L CNN
+F 1 "GND_" V 6445 10928 50  0000 L CNN
+F 2 "" H 6400 11050 50  0001 C CNN
+F 3 "" H 6400 11050 50  0001 C CNN
+	1    6400 11000
+	0    -1   -1   0
+$EndComp
+$Comp
+L power_ports:GND_ P?
+U 1 1 5FEC74D0
+P 10800 9950
+F 0 "P?" V 10754 9878 50  0000 L CNN
+F 1 "GND_" V 10845 9878 50  0000 L CNN
+F 2 "" H 10800 10000 50  0001 C CNN
+F 3 "" H 10800 10000 50  0001 C CNN
+	1    10800 9950
+	0    -1   -1   0
+$EndComp
+$Comp
+L power_ports:GND_ P?
+U 1 1 5FED26E6
+P 10750 13150
+F 0 "P?" V 10704 13078 50  0000 L CNN
+F 1 "GND_" V 10795 13078 50  0000 L CNN
+F 2 "" H 10750 13200 50  0001 C CNN
+F 3 "" H 10750 13200 50  0001 C CNN
+	1    10750 13150
+	0    -1   -1   0
+$EndComp
+$Comp
+L power_ports:GND_ P?
+U 1 1 5FEDD92A
+P 10700 14600
+F 0 "P?" V 10654 14528 50  0000 L CNN
+F 1 "GND_" V 10745 14528 50  0000 L CNN
+F 2 "" H 10700 14650 50  0001 C CNN
+F 3 "" H 10700 14650 50  0001 C CNN
+	1    10700 14600
+	0    -1   -1   0
+$EndComp
+$Comp
+L power_ports:GND_ P?
+U 1 1 5FEF19BD
+P 4100 6200
+F 0 "P?" V 4054 6128 50  0000 L CNN
+F 1 "GND_" V 4145 6128 50  0000 L CNN
+F 2 "" H 4100 6250 50  0001 C CNN
+F 3 "" H 4100 6250 50  0001 C CNN
+	1    4100 6200
+	0    -1   -1   0
+$EndComp
+Wire Wire Line
+	8950 7150 8950 7250
+Connection ~ 8950 7250
+Wire Wire Line
+	8950 7250 8950 7350
+Wire Wire Line
+	8950 5450 8950 5350
+$Comp
+L power_ports:GND_ P?
+U 1 1 5FF2E900
+P 9150 7250
+F 0 "P?" V 9104 7178 50  0000 L CNN
+F 1 "GND_" V 9195 7178 50  0000 L CNN
+F 2 "" H 9150 7300 50  0001 C CNN
+F 3 "" H 9150 7300 50  0001 C CNN
+	1    9150 7250
+	0    1    1    0
+$EndComp
+Wire Wire Line
+	7500 4750 7500 5750
+Wire Wire Line
+	4900 4750 7500 4750
+Wire Wire Line
+	7550 4800 4950 4800
+Wire Wire Line
+	7550 5650 7550 4800
+$Comp
+L MAX3523ETP_:MAX3523ETP+ U?
+U 1 1 5FEA0D8A
+P 8250 6450
+F 0 "U?" H 8250 7820 50  0000 C CNN
+F 1 "MAX3523ETP+" H 8250 7729 50  0000 C CNN
+F 2 "QFN65P500X500X80-21N" H 8250 6450 50  0001 L BNN
+F 3 "" H 8250 6450 50  0001 L BNN
+F 4 "QFN65P500X500X80-21N" H 8250 6450 50  0001 L BNN "Package"
+F 5 "Maxim Integrated" H 8250 6450 50  0001 L BNN "Manufacturer"
+	1    8250 6450
+	1    0    0    -1
+$EndComp
 $EndSCHEMATC

Commit message: work some more on schematic
Parts:
- removed J? (x3): 5-1814400-1, digikey-footprints:RF_SMA_RightAngle_5-1814400-1, symbol dk_Coaxial-Connectors-RF:5-1814400-1
- removed P? (x10): GND_, symbol power_ports:GND_
- removed U?: MAX3523ETP+, QFN65P500X500X80-21N, symbol MAX3523ETP_:MAX3523ETP+
- removed U? (x10): SKY13414-485LF, IC_SKY13414-485LF, symbol SKY13414-485LF:SKY13414-485LF
- added C? (x4): 0.1uF, CAPC2012X135N, symbol GRM21BR71C105KA01K:GRM21BR71C105KA01K
- added L?: LQH32DN150K53L, IND_LQH32DN150K53L, symbol LQH32DN150K53L:LQH32DN150K53L
- added P? (x4): GND_, symbol power_ports:GND_
- added R?: 1500, RESC2012X65N, symbol 9-2176091-2:9-2176091-2
- added T?: MABA-007159-000000, digikey-footprints:SMD-5-6_3.83x2.79mm, symbol dk_Balun:MABA-007159-000000
- added U?: PHA-13HLN+, symbol combo:PHA-13HLN+
- added U?: 0603CS-5N1XJLU, INDC1811X91N, symbol 0603CS-5N1XJLU:0603CS-5N1XJLU
Connections:
- net at U?.2 (RF1): now also T?.5
- net at U?.3 (RF2): now also T?.1
- new net: C?.1, C?.2, U?.1 (RF-IN)
- new net: P?.~, U?.2 (GND)
- new net: C?.1, L?.1, R?.2, U?.3 (RF-OUT_&_DC-IN)
- new net: C?.2, R?.1
- new net: C?.1, U?.1
- new net: C?.2, T?.3, U?.2
- new net: C?.1, P?.~
- new net: P?.~, T?.4

Commit message: add libs
Parts:
- removed J?: CX70M-24P1, digikey-footprints:USB-C_Female_CX70M-24P1, symbol dk_USB-DVI-HDMI-Connectors:CX70M-24P1
- removed P? (x3): GND_, symbol power_ports:GND_
- removed R? (x2): 5.1k, RESC2012X65N, symbol 9-2176091-2:9-2176091-2
- removed U?: Si514, symbol Si514:Si514
- added J?: 690-005-299-043, digikey-footprints:USB_Mini_B_Female_690-005-299-043, symbol dk_USB-DVI-HDMI-Connectors:690-005-299-043
- added J? (x2): 22-23-2021, digikey-footprints:PinHeader_1x2_P2.54mm_Drill1.02mm, symbol dk_Rectangular-Connectors-Headers-Male-Pins:22-23-2021
- added J? (x2): 142-0701-801, digikey-footprints:RF_SMA_BoardEdge_142-0701-801, symbol dk_Coaxial-Connectors-RF:142-0701-801
- added P? (x3): GND_, symbol power_ports:GND_
- added P?: +5v, symbol power_ports:+5v
- added T?: MABA-007159-000000, digikey-footprints:SMD-5-6_3.83x2.79mm, symbol dk_Balun:MABA-007159-000000
Connections:
- net at U?.100 (PA11): now also J?.2
- net at U?.101 (PA12): now also J?.1
- net at U?.4 (CLK+), U?.5 (LO1): now also U?.5 (LO1)
- net at U?.4 (LO2), U?.5 (CLK-): now also U?.4 (LO2)
- net at U?.2 (RF1): now also T?.5
- net at U?.3 (RF2): now also T?.1
- new net: P?.~, T?.4
- new net: J?.1, P?.~
- new net: J?.2, J?.2
- new net: J?.1, J?.3
- new net: J?.5, P?.~
- new net: J?.SH, P?.~

Commit message: add power to stm32
Parts:
- added J?: 22-23-2021, digikey-footprints:PinHeader_1x2_P2.54mm_Drill1.02mm, symbol dk_Rectangular-Connectors-Headers-Male-Pins:22-23-2021
- added P?: +3v, symbol power_ports:+3v
- added P?: GND_, symbol power_ports:GND_
Connections:
- net at P?.~, U?.104 (VSS), U?.118 (VSS)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: now also U?.14 (VSSSMPS), U?.15 (VLXSMPS), U?.17 (VFBSMPS), U?.34 (VSSA)
- net at U?.105 (VDDLDO): now also U?.106 (VDD), U?.119 (VDD), U?.129 (VDD), U?.13 (VDD), U?.143 (VDDLDO), U?.144 (VDD), U?.16 (VDDSMPS), U?.19 (VDD), U?.32 (VDD), U?.36 (VDDA), U?.42 (VDD), U?.56 (VDD), U?.7 (VDD), U?.70 (VDDLDO), U?.71 (VDD), U?.79 (VDD), U?.92 (VDD), P?.~
- net at U?.8 (VBAT): now also J?.2
- new net: J?.1, P?.~
Other:
- moved on the sheet: J?, U?, U?B, U?C

Commit message: annotate schematic
Parts:
- removed P? (x11): GND_, symbol power_ports:GND_
- removed P? (x2): +5v, symbol power_ports:+5v
- removed P? (x2): +3v, symbol power_ports:+3v
- gave numbers to parts that had none: 21
